Commit message: adding triton HIL to jackal

File: jackal_description/urdf/jackal.urdf.xacro (robot description, xacro)
@@ -228,3 +228,13 @@
   <!-- Optional for Clearpath internal softwares -->
   <xacro:include filename="$(optenv CPR_URDF_EXTRAS empty.urdf)" />
+  <!-- Triton model -->
+  <xacro:include filename="$(find accerion_triton_description)/urdf/triton_sensor.urdf.xacro"/>
+  <xacro:include filename="$(find thor_description)/urdf/triton_sensor_simulated.xacro" />
+  <xacro:triton_sensor_simulated name="triton"/>
+  <joint name="triton_mid_joint" type="fixed">
+    <origin xyz="0.2538 -0.0014 0" rpy="0 0 1.5691" />
+    <!-- <origin xyz="0.125 0.0 0.04" rpy="0 0 -${PI/2.0}"/> -->
+    <parent link="base_link"/>
+    <child link="triton_link"/>
+  </joint>
 </robot>

Commit message: fixed position of triton in urdf

File: jackal_description/urdf/jackal.urdf.xacro (robot description, xacro)
@@ -233,6 +233,5 @@
   <xacro:triton_sensor_simulated name="triton"/>
   <joint name="triton_mid_joint" type="fixed">
-    <origin xyz="0.2538 -0.0014 0" rpy="0 0 1.5691" />
-    <!-- <origin xyz="0.125 0.0 0.04" rpy="0 0 -${PI/2.0}"/> -->
+    <origin xyz="0.2538 0.0 -0.02" rpy="0.01 -0.005 -${PI/2.0}"/>
     <parent link="base_link"/>
     <child link="triton_link"/>
